File: Hardware/Basic/Top/SmartWatch-Basic-Top.brd (EAGLE design)
At the start: 38 x 38 mm, 44 parts, among them U2 NRF52832_MODULE_MDBT42

Commit message: top section
Parts:
- added C2: 1u, LinnesLab-Passives:C0603
- added R8, R9: 10k, LinnesLab-Passives:R0603
- added S1: (no value), switch-omron:B3F-10XX
- added U4: PCF8523, LinnesLab-Clocks:SO8
- added XTAL3: 32.7680kHz, LinnesLab-Clocks:2-SMD.NOLEAD.2.0MMTO1.2MM
- moved J2 24.7 mm to (1.80, 15.6), turned to 270 degrees
- moved U3 1.80 mm to (17.4, 21.3)
- moved USB2 1.27 mm to (2.08, 5.79), turned to 90 degrees
Connections:
- new net N$19: U4.2, XTAL3.P$1
- new net N$20: U4.1, XTAL3.P$2
- new net VBATT: U4.3
- net 3.3V: now also C2.1, R8.2, R9.2, U4.8
- net GND: now also C2.2, U4.4
- net SCL: now also R8.1, U4.6
- net SDA: now also R9.1, U4.5
