File: Hardware/Basic/Top/SmartWatch-Basic-Top.sch (EAGLE design)
At the start: 44 parts, among them U2 NRF52832_MODULE_MDBT42

Commit message: top section
Parts:
- added C2: 1u, LinnesLab-Passives:CAPACITOR0603
- added R8, R9: 10k, LinnesLab-Passives:RESISTOR0603
- added S1: (no value), switch-omron:10-XX
- added U4: PCF8523, LinnesLab-Clocks:PCF8523
- added XTAL3: 32.7680kHz, LinnesLab-Clocks:CRYSTALECS-.327-12.5-12-C-TR
Connections:
- new net N$19: U4.OSCO, XTAL3.1
- new net N$20: U4.OSCI, XTAL3.2
- new net VBATT: U4.VBAT
- net 3.3V: now also C2.1, R8.2, R9.2, U4.VDD
- net GND: now also C2.2, U4.VSS
- net SCL: now also R8.1, U4.SCL
- net SDA: now also R9.1, U4.SDA
Other:
- note added: "Back-up battery if desired"
- note added: "Buttons"
- note added: "Cortex Debugger/ Programmer"
- note added: "I2C Address = 0x68h"
- note added: "Power Management"
- note added: "RTC"
- note added: "Real-Time Clock"
- note added: "SD Card"
- note added: "nRF52832 Module"
- moved on the sheet: C14, C20, C21, C5, C6, CHRG2, D1, D4, D5, J2, LDO2, R11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
